Commit message: improvements of the repo.

File: URDFs/Robots/Universal_Robots_UR3/Universal_Robots_UR3.urdf (robot description, URDF)
Before this commit: robot Universal_Robots_UR3, 8 links, 7 joints
Links:
- removed link Base_Link
- added link Base_Link_1, mass 2.0; collision mesh filename=/Mesh/Collision/Base.stl; visual mesh filename=/Mesh/Visual/Base.stl
- link Link_1: mass 1.0 -> 2.0; geometry collision mesh filename=/Mesh/Collision/Joint_1.stl; visual mesh filename=/Mesh/Visual/Joint_1.stl
- link Link_2: mass 1.0 -> 3.42; geometry collision mesh filename=/Mesh/Collision/Joint_2.stl; visual mesh filename=/Mesh/Visual/Joint_2.stl
- link Link_3: mass 1.0 -> 1.26; geometry collision mesh filename=/Mesh/Collision/Joint_3.stl; visual mesh filename=/Mesh/Visual/Joint_3.stl
- link Link_4: mass 1.0 -> 0.8; geometry collision mesh filename=/Mesh/Collision/Joint_4.stl; visual mesh filename=/Mesh/Visual/Joint_4.stl
- link Link_5: mass 1.0 -> 0.8; geometry collision mesh filename=/Mesh/Collision/Joint_5.stl; visual mesh filename=/Mesh/Visual/Joint_5.stl
- link Link_6: mass 1.0 -> 0.35; geometry collision mesh filename=/Mesh/Collision/Joint_6.stl; visual mesh filename=/Mesh/Visual/Joint_6.stl
Joints:
- joint Joint_1: limit lower=-3.141592653589793 upper=3.141592653589793 effort=150.0 velocity=1.0 -> lower=-3.1415927410125732 upper=3.1415927410125732 effort=56.0 velocity=3.14; origin xyz=0.0 0.0 0.1519 rpy=0.0 0.0 0.0 -> xyz=0.0 0.0 0.15189999341964722 rpy=-0.0 0.0 -0.0; parent Base_Link -> Base_Link_1
- joint Joint_2: limit lower=-3.141592653589793 upper=3.141592653589793 effort=150.0 velocity=1.0 -> lower=-3.1415927410125732 upper=3.1415927410125732 effort=56.0 velocity=3.14; origin xyz=0.0 0.0 0.0 rpy=1.5707963267948966 0.0 0.0 -> xyz=0.0 0.0 0.0 rpy=1.5707963705062866 0.0 -0.0
- joint Joint_3: limit lower=-3.141592653589793 upper=3.141592653589793 effort=150.0 velocity=1.0 -> lower=-3.1415927410125732 upper=3.1415927410125732 effort=28.0 velocity=3.14; origin xyz=-0.24365 0.0 0.0 rpy=0.0 0.0 0.0 -> xyz=-0.24365000426769257 0.0 0.0 rpy=-0.0 0.0 -0.0
- joint Joint_4: limit lower=-3.141592653589793 upper=3.141592653589793 effort=150.0 velocity=1.0 -> lower=-3.1415927410125732 upper=3.1415927410125732 effort=12.0 velocity=6.28; origin xyz=-0.2132499 0.0 0.11235 rpy=0.0 0.0 0.0 -> xyz=-0.21324999630451202 0.0 0.11235000193119049 rpy=-0.0 0.0 -0.0
- joint Joint_5: limit lower=-3.141592653589793 upper=3.141592653589793 effort=150.0 velocity=1.0 -> lower=-3.1415927410125732 upper=3.1415927410125732 effort=12.0 velocity=6.28; origin xyz=0.0 -0.08535 0.0 rpy=1.5707963267948966 0.0 0.0 -> xyz=0.0 -0.08534999191761017 0.0 rpy=1.5707963705062866 0.0 -0.0
- joint Joint_6: limit lower=-3.141592653589793 upper=3.141592653589793 effort=150.0 velocity=1.0 -> lower=-3.1415927410125732 upper=3.1415927410125732 effort=12.0 velocity=6.28; origin xyz=0.0 0.0819 0.0 rpy=-1.5707963267948966 0.0 0.0 -> xyz=0.0 0.08190000057220459 -7.450580596923828e-09 rpy=-1.5707963705062866 0.0 -0.0

Commit message: improvements of the repo.

File: URDFs/Robots/Universal_Robots_UR3/Universal_Robots_UR3.urdf (robot description, URDF)
Before this commit: robot Universal_Robots_UR3, 8 links, 7 joints
Links:
- removed link Base_Link
- removed link EE_Link
- removed link Link_1
- removed link Link_2
- removed link Link_3
- removed link Link_4
- removed link Link_5
- removed link Link_6
- added link base_link, mass 2.0; collision mesh filename=/Mesh/Collision/Base.stl; visual mesh filename=/Mesh/Visual/Base.stl
- added link link_1, mass 1.26; collision mesh filename=/Mesh/Collision/Joint_1.stl; visual mesh filename=/Mesh/Visual/Joint_1.stl
- added link link_2, mass 1.26; collision mesh filename=/Mesh/Collision/Joint_2.stl; visual mesh filename=/Mesh/Visual/Joint_2.stl
- added link link_3, mass 1.26; collision mesh filename=/Mesh/Collision/Joint_3.stl; visual mesh filename=/Mesh/Visual/Joint_3.stl
- added link link_4, mass 1.26; collision mesh filename=/Mesh/Collision/Joint_4.stl; visual mesh filename=/Mesh/Visual/Joint_4.stl
- added link link_5, mass 1.26; collision mesh filename=/Mesh/Collision/Joint_5.stl; visual mesh filename=/Mesh/Visual/Joint_5.stl
- added link link_6, mass 1.26; collision mesh filename=/Mesh/Collision/Joint_6.stl; visual mesh filename=/Mesh/Visual/Joint_6.stl
- added link tool0_link
Joints:
- removed joint EE
- removed joint Joint_1
- removed joint Joint_2
- removed joint Joint_3
- removed joint Joint_4
- removed joint Joint_5
- removed joint Joint_6
- added joint joint_1: type revolute, parent base_link, child link_1, origin xyz=0.0 0.0 0.15190 rpy=0.0 0.0 0.0, axis 0 0 1, limit lower=-3.14159 upper=3.14159 effort=28.0 velocity=3.14
- added joint joint_2: type revolute, parent link_1, child link_2, origin xyz=0.0 0.0 0.0 rpy=1.57080 0.0 0.0, axis 0 0 1, limit lower=-3.14159 upper=3.14159 effort=28.0 velocity=3.14
- added joint joint_3: type revolute, parent link_2, child link_3, origin xyz=-0.24365 0.0 0.0 rpy=0.0 0.0 0.0, axis 0 0 1, limit lower=-3.14159 upper=3.14159 effort=28.0 velocity=3.14
- added joint joint_4: type revolute, parent link_3, child link_4, origin xyz=-0.21325 0.0 0.11235 rpy=0.0 0.0 0.0, axis 0 0 1, limit lower=-3.14159 upper=3.14159 effort=28.0 velocity=3.14
- added joint joint_5: type revolute, parent link_4, child link_5, origin xyz=0.0 -0.08535 0.0 rpy=1.57080 0.0 0.0, axis 0 0 1, limit lower=-3.14159 upper=3.14159 effort=28.0 velocity=3.14
- added joint joint_6: type revolute, parent link_5, child link_6, origin xyz=0.0 0.08190 0.0 rpy=-1.57080 0.0 0.0, axis 0 0 1, limit lower=-3.14159 upper=3.14159 effort=28.0 velocity=3.14
- added joint tool0: type fixed, parent link_3, child tool0_link, origin xyz=0.0 0.0 0.0 rpy=0.0 0.0 0.0

Commit message: improvements of the repo.

File: URDFs/Robots/Universal_Robots_UR3/Universal_Robots_UR3.urdf (robot description, URDF)
Before this commit: robot Universal_Robots_UR3, 8 links, 7 joints
Links:
- link base_link: geometry collision sphere radius=0.01; visual sphere radius=0.01
- link link_1: geometry collision sphere radius=0.01; visual sphere radius=0.01
- link link_2: geometry collision sphere radius=0.01; visual sphere radius=0.01
- link link_3: geometry collision sphere radius=0.01; visual sphere radius=0.01
- link link_4: geometry collision sphere radius=0.01; visual sphere radius=0.01
- link link_5: geometry collision sphere radius=0.01; visual sphere radius=0.01
- link link_6: geometry collision sphere radius=0.01; visual sphere radius=0.01
Joints:
- joint joint_1: axis 0 0 1 -> 0.0 0.0 1
- joint joint_2: axis 0 0 1 -> 0.0 0.0 1
- joint joint_3: axis 0 0 1 -> 0.0 0.0 1
- joint joint_4: axis 0 0 1 -> 0.0 0.0 1
- joint joint_5: axis 0 0 1 -> 0.0 0.0 1
- joint joint_6: axis 0 0 1 -> 0.0 0.0 1

Commit message: improvements of the repo.

File: URDFs/Robots/Universal_Robots_UR3/Universal_Robots_UR3.urdf (robot description, URDF)
Before this commit: robot Universal_Robots_UR3, 8 links, 7 joints
Links:
- link base_link: geometry collision mesh filename=/Mesh/Collision/Base.stl; visual mesh filename=/Mesh/Visual/Base.stl
- link link_1: mass 1.26 -> 2.0; geometry collision mesh filename=/Mesh/Collision/Joint_1.stl; visual mesh filename=/Mesh/Visual/Joint_1.stl
- link link_2: mass 1.26 -> 3.42; geometry collision mesh filename=/Mesh/Collision/Joint_2.stl; visual mesh filename=/Mesh/Visual/Joint_2.stl
- link link_3: geometry collision mesh filename=/Mesh/Collision/Joint_3.stl; visual mesh filename=/Mesh/Visual/Joint_3.stl
- link link_4: mass 1.26 -> 0.8; geometry collision mesh filename=/Mesh/Collision/Joint_4.stl; visual mesh filename=/Mesh/Visual/Joint_4.stl
- link link_5: mass 1.26 -> 0.8; geometry collision mesh filename=/Mesh/Collision/Joint_5.stl; visual mesh filename=/Mesh/Visual/Joint_5.stl
- link link_6: mass 1.26 -> 0.35; geometry collision mesh filename=/Mesh/Collision/Joint_6.stl; visual mesh filename=/Mesh/Visual/Joint_6.stl
Joints:
- joint joint_1: axis 0.0 0.0 1 -> 0 0 1; limit lower=-3.14159 upper=3.14159 effort=28.0 velocity=3.14 -> lower=-3.1415927410 upper=3.1415927410 effort=56.0 velocity=3.14; origin xyz=0.0 0.0 0.15190 rpy=0.0 0.0 0.0 -> xyz=0.0 0.0 0.1518999934 rpy=0.0 0.0 0.0
- joint joint_2: axis 0.0 0.0 1 -> 0 0 1; limit lower=-3.14159 upper=3.14159 effort=28.0 velocity=3.14 -> lower=-3.1415927410 upper=3.1415927410 effort=56.0 velocity=3.14; origin xyz=0.0 0.0 0.0 rpy=1.57080 0.0 0.0 -> xyz=0.0 0.0 0.0 rpy=1.5707999468 0.0 0.0
- joint joint_3: axis 0.0 0.0 1 -> 0 0 1; limit lower=-3.14159 upper=3.14159 effort=28.0 velocity=3.14 -> lower=-3.1415927410 upper=3.1415927410 effort=28.0 velocity=3.14; origin xyz=-0.24365 0.0 0.0 rpy=0.0 0.0 0.0 -> xyz=-0.2436500043 0.0 0.0 rpy=0.0 0.0 0.0
- joint joint_4: axis 0.0 0.0 1 -> 0 0 1; limit lower=-3.14159 upper=3.14159 effort=28.0 velocity=3.14 -> lower=-3.1415927410 upper=3.1415927410 effort=12.0 velocity=6.28; origin xyz=-0.21325 0.0 0.11235 rpy=0.0 0.0 0.0 -> xyz=-0.2132499963 0.0 0.1123500019 rpy=0.0 0.0 0.0
- joint joint_5: axis 0.0 0.0 1 -> 0 0 1; limit lower=-3.14159 upper=3.14159 effort=28.0 velocity=3.14 -> lower=-3.1415927410 upper=3.1415927410 effort=12.0 velocity=6.28; origin xyz=0.0 -0.08535 0.0 rpy=1.57080 0.0 0.0 -> xyz=0.0 -0.0853499994 0.0 rpy=1.5707999468 0.0 0.0
- joint joint_6: axis 0.0 0.0 1 -> 0 0 1; limit lower=-3.14159 upper=3.14159 effort=28.0 velocity=3.14 -> lower=-3.1415927410 upper=3.1415927410 effort=12.0 velocity=6.28; origin xyz=0.0 0.08190 0.0 rpy=-1.57080 0.0 0.0 -> xyz=0.0 0.0819000006 0.0 rpy=-1.5707999468 0.0 0.0
- joint tool0: parent link_3 -> link_6

Commit message: improvements of the repo.

File: URDFs/Robots/Universal_Robots_UR3/Universal_Robots_UR3.urdf (robot description, URDF)
Before this commit: robot Universal_Robots_UR3, 8 links, 7 joints
Joints:
- joint joint_1: origin xyz=0.0 0.0 0.1518999934 rpy=0.0 0.0 0.0 -> xyz=0.0 0.0 0.15190 rpy=0.0 0.0 0.0
- joint joint_3: origin xyz=-0.2436500043 0.0 0.0 rpy=0.0 0.0 0.0 -> xyz=-0.24365 0.0 0.0 rpy=0.0 0.0 0.0
- joint joint_4: origin xyz=-0.2132499963 0.0 0.1123500019 rpy=0.0 0.0 0.0 -> xyz=-0.21325 0.0 0.11235 rpy=0.0 0.0 0.0
- joint joint_5: origin xyz=0.0 -0.0853499994 0.0 rpy=1.5707999468 0.0 0.0 -> xyz=0.0 -0.08535 0.0 rpy=1.5707999468 0.0 0.0
- joint joint_6: origin xyz=0.0 0.0819000006 0.0 rpy=-1.5707999468 0.0 0.0 -> xyz=0.0 0.08190 0.0 rpy=-1.5707999468 0.0 0.0

Commit message: improvements of the repo.

File: URDFs/Robots/Universal_Robots_UR3/Universal_Robots_UR3.urdf (robot description, URDF)
Before this commit: robot Universal_Robots_UR3, 8 links, 7 joints
Links:
- link base_link: geometry collision sphere radius=0.01; visual sphere radius=0.01
- link link_1: geometry collision sphere radius=0.01; visual sphere radius=0.01
- link link_2: geometry collision sphere radius=0.01; visual sphere radius=0.01
- link link_3: geometry collision sphere radius=0.01; visual sphere radius=0.01
- link link_4: geometry collision sphere radius=0.01; visual sphere radius=0.01
- link link_5: geometry collision sphere radius=0.01; visual sphere radius=0.01
- link link_6: geometry collision sphere radius=0.01; visual sphere radius=0.01
