Commit message: improvements of the repo.

File: URDFs/Robots/ABB_IRB_120/ABB_IRB_120.urdf (robot description, URDF)
Before this commit: robot ABB_IRB_120, 8 links, 7 joints
Links:
- link base_link: geometry collision mesh filename=/Mesh/Collision/Base.stl; visual mesh filename=/Mesh/Visual/Base.stl
- link link_1: geometry collision mesh filename=/Mesh/Collision/Joint_1.stl; visual mesh filename=/Mesh/Visual/Joint_1.stl
- link link_2: geometry collision mesh filename=/Mesh/Collision/Joint_2.stl; visual mesh filename=/Mesh/Visual/Joint_2.stl
- link link_3: geometry collision mesh filename=/Mesh/Collision/Joint_3.stl; visual mesh filename=/Mesh/Visual/Joint_3.stl
- link link_4: geometry collision mesh filename=/Mesh/Collision/Joint_4.stl; visual mesh filename=/Mesh/Visual/Joint_4.stl
- link link_5: geometry collision mesh filename=/Mesh/Collision/Joint_5.stl; visual mesh filename=/Mesh/Visual/Joint_5.stl
- link link_6: geometry collision mesh filename=/Mesh/Collision/Joint_6.stl; visual mesh filename=/Mesh/Visual/Joint_6.stl

File: URDFs/Robots/Universal_Robots_UR3/Universal_Robots_UR3.urdf (robot description, URDF)
Before this commit: robot Universal_Robots_UR3, 8 links, 7 joints
Links:
- link base_link: geometry collision mesh filename=/Mesh/Collision/Base.stl; visual mesh filename=/Mesh/Visual/Base.stl
- link link_1: geometry collision mesh filename=/Mesh/Collision/Joint_1.stl; visual mesh filename=/Mesh/Visual/Joint_1.stl
- link link_2: geometry collision mesh filename=/Mesh/Collision/Joint_2.stl; visual mesh filename=/Mesh/Visual/Joint_2.stl
- link link_3: geometry collision mesh filename=/Mesh/Collision/Joint_3.stl; visual mesh filename=/Mesh/Visual/Joint_3.stl
- link link_4: geometry collision mesh filename=/Mesh/Collision/Joint_4.stl; visual mesh filename=/Mesh/Visual/Joint_4.stl
- link link_5: geometry collision mesh filename=/Mesh/Collision/Joint_5.stl; visual mesh filename=/Mesh/Visual/Joint_5.stl
- link link_6: geometry collision mesh filename=/Mesh/Collision/Joint_6.stl; visual mesh filename=/Mesh/Visual/Joint_6.stl

Commit message: improvements of the repo.

File: URDFs/Robots/ABB_IRB_120/ABB_IRB_120.urdf (robot description, URDF)
Before this commit: robot ABB_IRB_120, 8 links, 7 joints
Links:
- removed link tool0_link
- added link ee_link
- link base_link: geometry collision mesh filename=/Mesh/Visual/Base.stl; visual mesh filename=/Mesh/Visual/Base.stl
- link link_1: geometry collision mesh filename=/Mesh/Visual/Joint_1.stl; visual mesh filename=/Mesh/Visual/Joint_1.stl
- link link_2: geometry collision mesh filename=/Mesh/Visual/Joint_2.stl; visual mesh filename=/Mesh/Visual/Joint_2.stl
- link link_3: geometry collision mesh filename=/Mesh/Visual/Joint_3.stl; visual mesh filename=/Mesh/Visual/Joint_3.stl
- link link_4: geometry collision mesh filename=/Mesh/Visual/Joint_4.stl; visual mesh filename=/Mesh/Visual/Joint_4.stl
- link link_5: geometry collision mesh filename=/Mesh/Visual/Joint_5.stl; visual mesh filename=/Mesh/Visual/Joint_5.stl
- link link_6: geometry collision mesh filename=/Mesh/Visual/Joint_6.stl; visual mesh filename=/Mesh/Visual/Joint_6.stl
Joints:
- removed joint tool0
- added joint ee: type fixed, parent link_6, child ee_link, origin xyz=0.0 0.0 0.0 rpy=0.0 0.0 0.0
