Commit message: improvements of the repo.

File: URDFs/Viewpoint/Viewpoint.urdf (robot description, URDF)
Before this commit: robot Viewpoint, 4 links, 3 joints
Links:
- removed link Viewpoint_Link
- added link Base_Link; visual mesh filename=/Mesh/Visual/Viewpoint.stl scale=1 1 1
Joints:
- joint X_Axis: parent Viewpoint_Link -> Base_Link
- joint Y_Axis: parent Viewpoint_Link -> Base_Link
- joint Z_Axis: parent Viewpoint_Link -> Base_Link

Commit message: improvements of the repo.

File: URDFs/Viewpoint/Viewpoint.urdf (robot description, URDF)
Before this commit: robot Viewpoint, 4 links, 3 joints
Links:
- removed link Base_Link
- removed link X_Axis_Link
- removed link Y_Axis_Link
- removed link Z_Axis_Link
- added link base_link; visual mesh filename=/Mesh/Visual/Viewpoint.stl scale=1 1 1
- added link x_axis_link; visual mesh filename=/Mesh/Visual/X_Axis.stl
- added link y_axis_link; visual mesh filename=/Mesh/Visual/Y_Axis.stl
- added link z_axis_link; visual mesh filename=/Mesh/Visual/Z_Axis.stl
Joints:
- removed joint X_Axis
- removed joint Y_Axis
- removed joint Z_Axis
- added joint x_axis: type fixed, parent base_link, child x_axis_link
- added joint y_axis: type fixed, parent base_link, child y_axis_link
- added joint z_axis: type fixed, parent base_link, child z_axis_link
