Commit message: improvements of the repo.

File: URDFs/Mechanisms/SMC_LEFB25_14000/SMC_LEFB25_14000.urdf (robot description, URDF)
Before this commit: robot SMC_LEFB25_14000, 4 links, 3 joints
Links:
- link Base_Link: mass 1.0 -> 5.0
- link Link_L: mass 1.0 -> 0.5
- link Link_Shuttle: mass 1.0 -> 0.25
Joints:
- joint Joint_L: limit lower=0.0 upper=1.4 effort=0.0 velocity=1.0 -> lower=0.0 upper=1.4 effort=1.0 velocity=2.0
- joint Shuttle: limit lower=0.0 upper=0.0 effort=0.0 velocity=1.0 -> lower=0.0 upper=0.0 effort=0.0 velocity=0.0

File: src/Evaluation/URDF/output.urdf (robot description, URDF)
Before this commit: robot Universal_Robots_UR3, 8 links, 7 joints
Joints:
- joint Joint_1: limit lower=-3.1415927410125732 upper=3.1415927410125732 effort=1.0 velocity=1.0 -> lower=-3.1415927410125732 upper=3.1415927410125732 effort=0.0 velocity=1.0
- joint Joint_2: limit lower=-3.1415927410125732 upper=3.1415927410125732 effort=1.0 velocity=1.0 -> lower=-3.1415927410125732 upper=3.1415927410125732 effort=0.0 velocity=1.0
- joint Joint_3: limit lower=-3.1415927410125732 upper=3.1415927410125732 effort=1.0 velocity=1.0 -> lower=-3.1415927410125732 upper=3.1415927410125732 effort=0.0 velocity=1.0
- joint Joint_4: limit lower=-3.1415927410125732 upper=3.1415927410125732 effort=1.0 velocity=1.0 -> lower=-3.1415927410125732 upper=3.1415927410125732 effort=0.0 velocity=1.0
- joint Joint_5: limit lower=-3.1415927410125732 upper=3.1415927410125732 effort=1.0 velocity=1.0 -> lower=-3.1415927410125732 upper=3.1415927410125732 effort=0.0 velocity=1.0
- joint Joint_6: limit lower=-3.1415927410125732 upper=3.1415927410125732 effort=1.0 velocity=1.0 -> lower=-3.1415927410125732 upper=3.1415927410125732 effort=0.0 velocity=1.0

Commit message: improvements of the repo.

File: URDFs/Mechanisms/SMC_LEFB25_14000/SMC_LEFB25_14000.urdf (robot description, URDF)
Before this commit: robot SMC_LEFB25_14000, 4 links, 3 joints
Links:
- link Base_Link: geometry collision mesh filename=/Mesh/Collision/Base.stl; visual mesh filename=/Mesh/Visual/Base.stl
- link Link_L: geometry collision mesh filename=/Mesh/Collision/Joint_L.stl; visual mesh filename=/Mesh/Visual/Joint_L.stl
- link Link_Shuttle: geometry collision mesh filename=/Mesh/Collision/Shuttle.stl; visual mesh filename=/Mesh/Visual/Shuttle.stl

Commit message: improvements of the repo.

File: URDFs/Mechanisms/SMC_LEFB25_14000/SMC_LEFB25_14000.urdf (robot description, URDF)
Before this commit: robot SMC_LEFB25_14000, 4 links, 3 joints
Links:
- removed link Base_Link
- removed link EE_Link
- removed link Link_L
- removed link Link_Shuttle
- added link base_link, mass 5.0; collision mesh filename=/Mesh/Collision/Base.stl; visual mesh filename=/Mesh/Visual/Base.stl
- added link ee_link
- added link link_L, mass 0.5; collision mesh filename=/Mesh/Collision/Joint_L.stl; visual mesh filename=/Mesh/Visual/Joint_L.stl
- added link link_Shuttle, mass 0.25; collision mesh filename=/Mesh/Collision/Shuttle.stl; visual mesh filename=/Mesh/Visual/Shuttle.stl
Joints:
- removed joint EE
- removed joint Joint_L
- removed joint Shuttle
- added joint ee: type fixed, parent link_shuttle, child ee_link, origin xyz=0.0 0.0 0.019998 rpy=0.0 0.0 0.0
- added joint joint_L: type prismatic, parent base_link, child link_L, origin xyz=0.0 0.0 0.168499 rpy=0.0 0.0 0.0, axis 0 1 0, limit lower=0.0 upper=1.4 effort=1.0 velocity=2.0
- added joint shuttle: type fixed, parent link_L, child link_shuttle, origin xyz=0.0 0.0 0.0 rpy=0.0 0.0 0.0, axis 0 1 0, limit lower=0.0 upper=0.0 effort=0.0 velocity=0.0

File: URDFs/Robots/ABB_IRB_120_L_Ax/ABB_IRB_120_L_Ax.urdf (robot description, URDF)
Before this commit: robot ABB_IRB_120_L_Ax, 9 links, 8 joints
Links:
- added link link_1, mass 3.45; collision mesh filename=/Mesh/Visual/Joint_1.stl; visual mesh filename=/Mesh/Visual/Joint_1.stl
- link base_link_1: mass 3.45 -> 8.25; geometry collision mesh filename=/Mesh/Visual/Base_1.stl; visual mesh filename=/Mesh/Visual/Base_1.stl
Joints:
- added joint base_1: type fixed, parent link_L, child base_link_1, origin xyz=0.0 0.0 0.0 rpy=0.0 0.0 0.0
- joint ee: parent link_7 -> link_6
- joint joint_1: child base_link_1 -> link_1; parent link_L -> base_link_1
- joint joint_2: parent link_0 -> link_1
- joint joint_3: parent link_1 -> link_2
- joint joint_4: parent link_2 -> link_3
- joint joint_5: parent link_3 -> link_4
- joint joint_6: parent link_4 -> link_5

Commit message: Update SMC_LEFB25_14000.urdf

File: URDFs/Mechanisms/SMC_LEFB25_14000/SMC_LEFB25_14000.urdf (robot description, URDF)
Before this commit: robot SMC_LEFB25_14000, 4 links, 3 joints
Links:
- removed link link_Shuttle
- added link link_shuttle, mass 0.25; collision mesh filename=/Mesh/Collision/Shuttle.stl; visual mesh filename=/Mesh/Visual/Shuttle.stl
